File: swadge-programmer/swadge-programmer.kicad_pcb (KiCad board)
At the start: 2 copper layers, 73.7 x 73.7 mm, 28 parts, among them J1 USB_B_Micro, J2 Conn_02x15_Top_Bottom, J3 Conn_02x15_Top_Bottom, J4 ftdi-header, J5 Conn_01x03_Male, SW1 4-1437565-2, SW2 4-1437565-2, SW3 4-1437565-2, SW4 SW_DPDT_x2, SW5 SW_DPDT_x2, U1 BUS_PCIexpress, U2 CP2102N-A01-GQFN24

Commit message: Move and reroute programmer
Parts:
- removed the svg2mod at (123.0, 64.0)
- moved R4 50.1 mm to (170.5, 85.0)
- moved R5 50.1 mm to (120.4, 85.0)
- moved J2 35.6 mm to (163.6, 87.0), turned to 270 degrees
- moved J3 35.6 mm to (163.6, 93.2), turned to 270 degrees
- moved SW1 17.3 mm to (171.2, 113.8)
- moved SW3 17.3 mm to (153.9, 113.8), turned to 270 degrees
- moved U1 15.6 mm to (163.1, 75.8), turned to 180 degrees
- moved C3 6.48 mm to (156.2, 61.0)
- moved R2 4.22 mm to (156.2, 65.5), turned to 180 degrees
- moved R1 3.86 mm to (156.2, 64.0), turned to 0 degrees
- moved R3 3.76 mm to (156.2, 67.1), turned to 180 degrees
- moved D1 3.53 mm to (166.2, 58.9)
- moved C1 2.91 mm to (160.1, 59.4)
- moved svg2mod 2.02 mm to (127.0, 54.0)
- moved C2 0.59 mm to (158.6, 59.4)
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Routing:
- net +3V3: track 123.2 -> 91.0 mm
- net 5V: track 64.3 -> 33.6 mm
- net Net-(R5-Pad1): track 24.6 -> 44.4 mm, vias 0 -> 1
- net Net-(C3-Pad1): track 55.3 -> 36.7 mm, vias 4 -> 2
- net RX: track 62.2 -> 80.3 mm, vias 0 -> 2
- net Net-(R4-Pad1): track 31.6 -> 13.6 mm, vias 1 -> 0
- net SW4: track 24.4 -> 41.7 mm
- net SW5: track 23.5 -> 40.3 mm
- net AUD_PWR: track 20.7 -> 37.3 mm
- net REST: track 20.8 -> 37.0 mm
- net _RES: track 73.5 -> 57.7 mm, vias 1 -> 0
- net TX: track 60.5 -> 76.1 mm
- net ADC_PIN: track 22.8 -> 38.0 mm
- net SW3: track 22.5 -> 37.6 mm
- net SW2: track 21.0 -> 34.3 mm
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Other:
- board text added: "Swadge Programmer 2.1.0"
- board text removed: "Swadge Programmer 2.0.0"
