File: swadge-programmer/swadge-programmer.kicad_pcb (KiCad board)
At the start: 2 copper layers, 73.7 x 73.7 mm, 28 parts, among them J1 USB_B_Micro, J2 Conn_02x15_Top_Bottom, J3 Conn_02x15_Top_Bottom, J4 ftdi-header, J5 Conn_01x03_Male, J6 Conn_01x03_Male, SW1 4-1437565-2, SW2 4-1437565-2, SW3 4-1437565-2, SW4 SW_DPDT_x2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

Commit message: Added signature
Other:
- board text added: "AEF'21"
